File: FlatSatModule.sch (KiCad schematic (older format))
At the start: 6 parts, among them J1 HEADER_13x2, J101 DB26_Male_HighDensity_Mountin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, J2 Micro_SD_Card_Det

Commit message: ?
Parts:
- added R1, R2: R, Resistor_SMD:R_0603_1608Metric_Pad1.05x0.95mm_HandSolder, symbol Device:R
- stm32101: footprint stm32:stm32f429i-disco -> Varistor:RV_Disc_D15.5mm_W8mm_P7.5mm
Connections:
- net labels added: SD_DET
- wire segments 32 -> 40
Changed lines of the file:
@@
 F 0 "stm32101" H 2425 7597 60  0000 C CNN
 F 1 "STM32F429i-Discovery" H 2425 7491 60  0000 C CNN
-F 2 "stm32:stm32f429i-disco" H 2525 6450 60  0001 C CNN
+F 2 "Varistor:RV_Disc_D15.5mm_W8mm_P7.5mm" H 2525 6450 60  0001 C CNN
 F 3 "" H 2525 6450 60  0000 C CNN
 	1    2425 5800
@@
 F 0 "stm32101" H 5550 7597 60  0000 C CNN
 F 1 "STM32F429i-Discovery" H 5550 7491 60  0000 C CNN
-F 2 "stm32:stm32f429i-disco" H 5650 6450 60  0001 C CNN
+F 2 "Varistor:RV_Disc_D15.5mm_W8mm_P7.5mm" H 5650 6450 60  0001 C CNN
 F 3 "" H 5650 6450 60  0000 C CNN
 	2    5550 5800
@@
 	1    0    0    -1
 $EndComp
+$Comp
+L Device:R R1
+U 1 1 5EFB0FAC
+P 8250 5000
+F 0 "R1" V 8043 5000 50  0000 C CNN
+F 1 "R" V 8134 5000 50  0000 C CNN
+F 2 "Resistor_SMD:R_0603_1608Metric_Pad1.05x0.95mm_HandSolder" V 8180 5000 50  0001 C CNN
+F 3 "~" H 8250 5000 50  0001 C CNN
+	1    8250 5000
+	0    1    1    0
+$EndComp
+$Comp
+L Device:R R2
+U 1 1 5EFB1F58
+P 8300 5550
+F 0 "R2" V 8093 5550 50  0000 C CNN
+F 1 "R" V 8184 5550 50  0000 C CNN
+F 2 "Resistor_SMD:R_0603_1608Metric_Pad1.05x0.95mm_HandSolder" V 8230 5550 50  0001 C CNN
+F 3 "~" H 8300 5550 50  0001 C CNN
+	1    8300 5550
+	0    1    1    0
+$EndComp
+Text Label 9350 5000 0    50   ~ 0
+VCC
+Wire Wire Line
+	8700 5550 8450 5550
+Wire Wire Line
+	8700 5000 8400 5000
+$Comp
+L power:GND #PWR0101
+U 1 1 5EFB5C13
+P 7650 5750
+F 0 "#PWR0101" H 7650 5500 50  0001 C CNN
+F 1 "GND" H 7655 5577 50  0000 C CNN
+F 2 "" H 7650 5750 50  0001 C CNN
+F 3 "" H 7650 5750 50  0001 C CNN
+	1    7650 5750
+	1    0    0    -1
+$EndComp
+Wire Wire Line
+	8100 5000 7650 5000
+Wire Wire Line
+	8150 5550 7650 5550
+Wire Wire Line
+	7650 5000 7650 5550
+Connection ~ 7650 5550
+Wire Wire Line
+	7650 5550 7650 5750
+Wire Wire Line
+	9350 5000 9000 5000
+Text Label 8200 3600 2    50   ~ 0
+VCC
+Text Label 8200 3700 2    50   ~ 0
+SD_DET
+Text Label 9350 5550 0    50   ~ 0
+SD_DET
+Wire Wire Line
+	9350 5550 9000 5550
 $EndSCHEMATC

Commit message: updated wiring + wired SD card
Parts:
- removed J1: HEADER_13x2, Connector_PinHeader_2.54mm:PinHeader_2x13_P2.54mm_Vertical, symbol w_connectors:HEADER_13x2
- removed J101: DB26_Male_HighDensity_MountingHoles, Connector_Dsub:DSUB-26-HD_Female_Horizontal_P2.29x1.98mm_EdgePinOffset8.35mm_Housed_MountingHolesOffset10.89mm, symbol db26hd:DB26_Male_HighDensity_MountingHoles
- added J1: DB15_Female_HighDensity, Connector_Dsub:DSUB-15-HD_Female_Horizontal_P2.29x2.54mm_EdgePinOffset9.40mm, symbol Connector:DB15_Female_HighDensity
- added J3: HEADER_15, Connector_PinHeader_1.27mm:PinHeader_1x15_P1.27mm_Vertical, symbol w_connectors:HEADER_15
- stm32101: footprint Varistor:RV_Disc_D15.5mm_W8mm_P7.5mm -> stm32:stm32f429i-disco
Connections:
- net labels added: BOOT0, I2C2_SCL, I2C2_SDA, I2C2_SDL, NC, NRST, PA0, PA1, PA10, PA11, PA12, PA13, PA14, PA15, PA2, PA3, PA4, PA5, PA6, PA7, PA8, PA9, PB0, PB1, PB10, PB11, PB12, PB13, PB14, PB15, PB2, PB3, PB4, PB5, PB6, PB7, PB8, PB9, PC0, PC1, PC10, PC11, PC12, PC13, PC14, PC15, PC2, PC3, PC4, PC5, PC6, PC7, PC8, PC9, PD0, PD1, PD10, PD11, PD12, PD13, PD14, PD15, PD2, PD3, PD4, PD5, PD6, PD7, PD8, PD9, PE0, PE1, PE10, PE11, PE12, PE13, PE14, PE15, PE2, PE3, PE4, PE5, PE6, PE7, PE8, PE9, PF0, PF1, PF10, PF11, PF12, PF13, PF14, PF15, PF2, PF3, PF4, PF5, PF6, PF7, PF8, PF9, PG0, PG1, PG10, PG11, PG12, PG13, PG14, PG15, PG2, PG3, PG4, PG5, PG6, PG7, PG8, PG9, PH0, PH1, SDIO_CK, SDIO_CMD, SD_CLK, SD_CMD, SD_D0, SD_D1, SD_D2, SD_D3, SD_DETA, SD_DETB, SD_VDD, SD_VSS, SPI1_MISO, SPI1_MOSI, SPI1_SCK, VCC3, VCC5, VDD
- net labels removed: CAN1_H, CAN1_L, I2C3_SCL, I2C3_SDA, SPI4_SS, UART2_RX, UART2_TX
- wire segments 40 -> 28
Other:
- moved on the sheet: stm32101A, stm32101B

Commit message: add USARTs and gnd plane filling
Parts:
- removed J1: DB15_Female_HighDensity, Connector_Dsub:DSUB-15-HD_Female_Horizontal_P2.29x2.54mm_EdgePinOffset9.40mm, symbol Connector:DB15_Female_HighDensity
- removed J3: HEADER_15, Connector_PinHeader_1.27mm:PinHeader_1x15_P1.27mm_Vertical, symbol w_connectors:HEADER_15
- added J1: DB26_Male_HighDensity_MountingHoles, Connector_Dsub:DSUB-26-HD_Male_Horizontal_P2.29x1.98mm_EdgePinOffset8.35mm_Housed_MountingHolesOffset10.89mm, symbol db26hd:DB26_Male_HighDensity_MountingHoles
- added J3: HEADER_13x2, Connector_PinHeader_2.54mm:PinHeader_2x13_P2.54mm_Vertical, symbol w_connectors:HEADER_13x2
Connections:
- net labels added: CAN1_RX, CAN1_TX, UART1_RX, UART1_TX, UART2_RX, UART2_TX
- wire segments 28 -> 34
Changed lines of the file:
@@
 Wire Wire Line
 	9350 5550 9000 5550
-$Comp
-L Connector:DB15_Female_HighDensity J1
-U 1 1 5F055F05
-P 1400 1750
-F 0 "J1" H 1400 2617 50  0000 C CNN
-F 1 "DB15_Female_HighDensity" H 1400 2526 50  0000 C CNN
-F 2 "Connector_Dsub:DSUB-15-HD_Female_Horizontal_P2.29x2.54mm_EdgePinOffset9.40mm" H 450 2150 50  0001 C CNN
-F 3 " ~" H 450 2150 50  0001 C CNN
-	1    1400 1750
-	1    0    0    -1
-$EndComp
-$Comp
-L w_connectors:HEADER_15 J3
-U 1 1 5F0575DD
-P 3500 1550
-F 0 "J3" H 3628 1603 60  0000 L CNN
-F 1 "HEADER_15" H 3628 1497 60  0000 L CNN
-F 2 "Connector_PinHeader_1.27mm:PinHeader_1x15_P1.27mm_Vertical" H 3500 1550 60  0001 C CNN
-F 3 "" H 3500 1550 60  0000 C CNN
-	1    3500 1550
-	1    0    0    -1
-$EndComp
 Text Label 5050 4100 2    50   ~ 0
 VCC3
@@
 Text Label 5400 2450 0    50   ~ 0
 SDIO_CK
-Text Label 1100 2150 2    50   ~ 0
+Text Label 1300 2550 2    50   ~ 0
 I2C1_SDA
-Text Label 1700 2150 0    50   ~ 0
+Text Label 1900 2450 0    50   ~ 0
 I2C1_SCL
-Text Label 1100 2050 2    50   ~ 0
+Text Label 1300 2450 2    50   ~ 0
 I2C2_SDA
-Text Label 1700 1950 0    50   ~ 0
+Text Label 1900 2250 0    50   ~ 0
 I2C2_SCL
-Text Label 1100 1950 2    50   ~ 0
+Text Label 1300 2350 2    50   ~ 0
 SPI1_SCK
-Text Label 1100 1850 2    50   ~ 0
+Text Label 1300 2250 2    50   ~ 0
 SPI1_MISO
-Text Label 1100 1750 2    50   ~ 0
+Text Label 1300 2150 2    50   ~ 0
 SPI1_MOSI
-Text Label 1700 1750 0    50   ~ 0
+Text Label 1900 2050 0    50   ~ 0
 SPI4_SCK
-Text Label 1100 1650 2    50   ~ 0
+Text Label 1300 2050 2    50   ~ 0
 SPI4_MISO
-Text Label 1700 1550 0    50   ~ 0
+Text Label 1900 1850 0    50   ~ 0
 SPI4_MOSI
-Text Label 3400 2250 2    50   ~ 0
+Text Label 3575 2200 2    50   ~ 0
 I2C1_SDA
-Text Label 3400 2150 2    50   ~ 0
+Text Label 3575 2100 2    50   ~ 0
 I2C1_SCL
-Text Label 3400 2050 2    50   ~ 0
+Text Label 3875 2100 0    50   ~ 0
 I2C2_SDA
-Text Label 3400 1950 2    50   ~ 0
+Text Label 3875 2200 0    50   ~ 0
 I2C2_SDL
-Text Label 3400 1850 2    50   ~ 0
+Text Label 3575 2000 2    50   ~ 0
 SPI1_SCK
-Text Label 3400 1750 2    50   ~ 0
+Text Label 3575 1900 2    50   ~ 0
 SPI1_MISO
-Text Label 3400 1650 2    50   ~ 0
+Text Label 3575 1800 2    50   ~ 0
 SPI1_MOSI
-Text Label 3400 1550 2    50   ~ 0
+Text Label 3875 1800 0    50   ~ 0
 SPI4_SCK
-Text Label 3400 1450 2    50   ~ 0
+Text Label 3875 1900 0    50   ~ 0
 SPI4_MISO
-Text Label 3400 1350 2    50   ~ 0
+Text Label 3875 2000 0    50   ~ 0
 SPI4_MOSI
 Text Label 8200 3300 2    50   ~ 0
@@
 GND
 $Comp
-L power:GND #PWR?
+L power:GND #PWR0101
 U 1 1 5F0DE653
 P 5175 900
-F 0 "#PWR?" H 5175 650 50  0001 C CNN
+F 0 "#PWR0101" H 5175 650 50  0001 C CNN
 F 1 "GND" V 5180 772 50  0000 R CNN
 F 2 "" H 5175 900 50  0001 C CNN
@@
 $EndComp
 $Comp
-L power:VCC #PWR?
+L power:VCC #PWR0102
 U 1 1 5F0DFC60
 P 5175 775
-F 0 "#PWR?" H 5175 625 50  0001 C CNN
+F 0 "#PWR0102" H 5175 625 50  0001 C CNN
 F 1 "VCC" V 5193 902 50  0000 L CNN
 F 2 "" H 5175 775 50  0001 C CNN
@@
 	5175 775  5375 775
 Text Label 5375 775  0    50   ~ 0
-VCC3
+VCC5
+Wire Wire Line
+	6175 1150 6375 1150
+Text Label 6175 1150 2    50   ~ 0
+PA11
+Text Label 6375 1150 0    50   ~ 0
+CAN1_RX
+Wire Wire Line
+	6175 1250 6375 1250
+Text Label 6175 1250 2    50   ~ 0
+PA12
+Text Label 6375 1250 0    50   ~ 0
+CAN1_TX
+Text Label 1300 1950 2    50   ~ 0
+CAN1_RX
+Text Label 1300 1850 2    50   ~ 0
+CAN1_TX
+Text Label 3575 1700 2    50   ~ 0
+CAN1_RX
+Text Label 3575 1600 2    50   ~ 0
+CAN1_TX
+Text Label 6375 1475 0    50   ~ 0
+UART1_TX
+Text Label 6175 1475 2    50   ~ 0
+PA9
+Wire Wire Line
+	6175 1475 6375 1475
+Text Label 6375 1375 0    50   ~ 0
+UART1_RX
+Text Label 6175 1375 2    50   ~ 0
+PA10
+Wire Wire Line
+	6175 1375 6375 1375
+Text Label 6375 1700 0    50   ~ 0
+UART2_TX
+Text Label 6175 1700 2    50   ~ 0
+PA2
+Text Label 6375 1600 0    50   ~ 0
+UART2_RX
+Text Label 6175 1600 2    50   ~ 0
+PA3
+Wire Wire Line
+	6175 1600 6375 1600
+Wire Wire Line
+	6175 1700 6375 1700
+Text Label 1900 1650 0    50   ~ 0
+UART1_RX
+Text Label 1300 1750 2    50   ~ 0
+UART1_TX
+Text Label 3875 1600 0    50   ~ 0
+UART1_RX
+Text Label 3875 1700 0    50   ~ 0
+UART1_TX
+$Comp
+L db26hd:DB26_Male_HighDensity_MountingHoles J1
+U 1 1 5F0EE44F
+P 1600 2150
+F 0 "J1" H 1600 3767 50  0000 C CNN
+F 1 "DB26_Male_HighDensity_MountingHoles" H 1600 3676 50  0000 C CNN
+F 2 "Connector_Dsub:DSUB-26-HD_Male_Horizontal_P2.29x1.98mm_EdgePinOffset8.35mm_Housed_MountingHolesOffset10.89mm" H 650 2550 50  0001 C CNN
+F 3 " ~" H 650 2550 50  0001 C CNN
+	1    1600 2150
+	1    0    0    -1
+$EndComp
+$Comp
+L w_connectors:HEADER_13x2 J3
+U 1 1 5F0FC4D0
+P 3725 1600
+F 0 "J3" H 3725 2437 60  0000 C CNN
+F 1 "HEADER_13x2" H 3725 2331 60  0000 C CNN
+F 2 "Connector_PinHeader_2.54mm:PinHeader_2x13_P2.54mm_Vertical" H 3725 1600 60  0001 C CNN
+F 3 "" H 3725 1600 60  0000 C CNN
+	1    3725 1600
+	1    0    0    -1
+$EndComp
+Text Label 1300 1550 2    50   ~ 0
+UART2_TX
+Text Label 1300 1650 2    50   ~ 0
+UART2_RX
+Text Label 3575 1500 2    50   ~ 0
+UART2_TX
+Text Label 3575 1400 2    50   ~ 0
+UART2_RX
+Text Label 1300 850  2    50   ~ 0
+VCC
+Text Label 1300 950  2    50   ~ 0
+GND
+Text Label 1600 2850 3    50   ~ 0
+GND
 $EndSCHEMATC

Commit message: Add SS for SPI buses
Connections:
- net labels added: SPI1_SS, SPI4_SS
- wire segments 34 -> 36
- no-connect marks 0 -> 4
Changed lines of the file:
@@
 Text Label 5050 7100 2    50   ~ 0
 PG3
-Text Label 6050 4100 0    50   ~ 0
-VCC3
 Text Label 6050 4200 0    50   ~ 0
 NC
@@
 SPI1_MOSI
 Wire Wire Line
-	5200 2000 5400 2000
-Text Label 5200 2000 2    50   ~ 0
-PE2
-Text Label 5400 2000 0    50   ~ 0
-SPI4_SCK
-Wire Wire Line
 	5200 2100 5400 2100
 Text Label 5200 2100 2    50   ~ 0
-PE5
+PE2
 Text Label 5400 2100 0    50   ~ 0
-SPI4_MISO
+SPI4_SCK
 Wire Wire Line
 	5200 2200 5400 2200
 Text Label 5200 2200 2    50   ~ 0
+PE5
+Text Label 5400 2200 0    50   ~ 0
+SPI4_MISO
+Wire Wire Line
+	5200 2300 5400 2300
+Text Label 5200 2300 2    50   ~ 0
 PE6
-Text Label 5400 2200 0    50   ~ 0
+Text Label 5400 2300 0    50   ~ 0
 SPI4_MOSI
 Wire Wire Line
-	5200 2350 5400 2350
-Text Label 5200 2350 2    50   ~ 0
+	5200 2550 5400 2550
+Text Label 5200 2550 2    50   ~ 0
 PD2
-Text Label 5400 2350 0    50   ~ 0
+Text Label 5400 2550 0    50   ~ 0
 SDIO_CMD
 Wire Wire Line
-	5200 2450 5400 2450
-Text Label 5200 2450 2    50   ~ 0
+	5200 2650 5400 2650
+Text Label 5200 2650 2    50   ~ 0
 PC12
-Text Label 5400 2450 0    50   ~ 0
+Text Label 5400 2650 0    50   ~ 0
 SDIO_CK
 Text Label 1300 2550 2    50   ~ 0
@@
 Text Label 1900 2050 0    50   ~ 0
 SPI4_SCK
-Text Label 1300 2050 2    50   ~ 0
+Text Label 1300 1950 2    50   ~ 0
 SPI4_MISO
 Text Label 1900 1850 0    50   ~ 0
@@
 SD_DETB
 Wire Wire Line
-	5200 2550 5400 2550
-Text Label 5200 2550 2    50   ~ 0
-PC8
-Text Label 5400 2550 0    50   ~ 0
-SD_D0
-Wire Wire Line
-	5200 2650 5400 2650
-Text Label 5200 2650 2    50   ~ 0
-PC9
-Text Label 5400 2650 0    50   ~ 0
-SD_D1
-Wire Wire Line
 	5200 2750 5400 2750
 Text Label 5200 2750 2    50   ~ 0
-PC10
+PC8
 Text Label 5400 2750 0    50   ~ 0
-SD_D2
+SD_D0
 Wire Wire Line
 	5200 2850 5400 2850
 Text Label 5200 2850 2    50   ~ 0
+PC9
+Text Label 5400 2850 0    50   ~ 0
+SD_D1
+Wire Wire Line
+	5200 2950 5400 2950
+Text Label 5200 2950 2    50   ~ 0
+PC10
+Text Label 5400 2950 0    50   ~ 0
+SD_D2
+Wire Wire Line
+	5200 3050 5400 3050
+Text Label 5200 3050 2    50   ~ 0
 PC11
-Text Label 5400 2850 0    50   ~ 0
+Text Label 5400 3050 0    50   ~ 0
 SD_D3
 Text Label 5050 7200 2    50   ~ 0
 GND
-Text Label 6050 7200 0    50   ~ 0
-GND
 Text Label 5050 5500 2    50   ~ 0
 GND
 Text Label 5050 4600 2    50   ~ 0
-GND
-Text Label 1725 7200 2    50   ~ 0
 GND
 Text Label 2725 7200 0    50   ~ 0
@@
 Text Label 1725 4200 2    50   ~ 0
 PF4
-Text Label 1725 4100 2    50   ~ 0
-VCC5
 Text Label 2725 7100 0    50   ~ 0
 PG4
@@
 $EndComp
 Wire Wire Line
-	5200 2950 5400 2950
-Text Label 5200 2950 2    50   ~ 0
-VCC3
-Text Label 5400 2950 0    50   ~ 0
-SD_DETA
-Wire Wire Line
-	5200 3050 5400 3050
-Text Label 5200 3050 2    50   ~ 0
-SD_DET
-Text Label 5400 3050 0    50   ~ 0
-SD_DETB
-Wire Wire Line
 	5200 3150 5400 3150
 Text Label 5200 3150 2    50   ~ 0
-GND
+VCC3
 Text Label 5400 3150 0    50   ~ 0
-SD_VSS
+SD_DETA
 Wire Wire Line
 	5200 3250 5400 3250
 Text Label 5200 3250 2    50   ~ 0
+SD_DET
+Text Label 5400 3250 0    50   ~ 0
+SD_DETB
+Wire Wire Line
+	5200 3350 5400 3350
+Text Label 5200 3350 2    50   ~ 0
+GND
+Text Label 5400 3350 0    50   ~ 0
+SD_VSS
+Wire Wire Line
+	5200 3450 5400 3450
+Text Label 5200 3450 2    50   ~ 0
 VCC3
-Text Label 5400 3250 0    50   ~ 0
+Text Label 5400 3450 0    50   ~ 0
 SD_VDD
 Text Label 7650 5000 2    50   ~ 0
@@
 Text Label 6375 1250 0    50   ~ 0
 CAN1_TX
-Text Label 1300 1950 2    50   ~ 0
+Text Label 1300 1750 2    50   ~ 0
 CAN1_RX
-Text Label 1300 1850 2    50   ~ 0
+Text Label 1300 1650 2    50   ~ 0
 CAN1_TX
-Text Label 3575 1700 2    50   ~ 0
+Text Label 3575 1600 2    50   ~ 0
 CAN1_RX
-Text Label 3575 1600 2    50   ~ 0
+Text Label 3575 1500 2    50   ~ 0
 CAN1_TX
 Text Label 6375 1475 0    50   ~ 0
@@
 Text Label 1900 1650 0    50   ~ 0
 UART1_RX
-Text Label 1300 1750 2    50   ~ 0
+Text Label 1300 1550 2    50   ~ 0
 UART1_TX
+Text Label 3875 1500 0    50   ~ 0
+UART1_RX
 Text Label 3875 1600 0    50   ~ 0
-UART1_RX
-Text Label 3875 1700 0    50   ~ 0
 UART1_TX
 $Comp
@@
 	1    0    0    -1
 $EndComp
-Text Label 1300 1550 2    50   ~ 0
+Text Label 1300 1450 2    50   ~ 0
+UART2_RX
+Text Label 3575 1400 2    50   ~ 0
 UART2_TX
-Text Label 1300 1650 2    50   ~ 0
-UART2_RX
-Text Label 3575 1500 2    50   ~ 0
-UART2_TX
-Text Label 3575 1400 2    50   ~ 0
+Text Label 3575 1300 2    50   ~ 0
 UART2_RX
 Text Label 1300 850  2    50   ~ 0
@@
 Text Label 1600 2850 3    50   ~ 0
 GND
+Wire Wire Line
+	5200 1950 5400 1950
+Text Label 5200 1950 2    50   ~ 0
+PA4
+Text Label 5400 1950 0    50   ~ 0
+SPI1_SS
+Wire Wire Line
+	5200 2400 5400 2400
+Text Label 5200 2400 2    50   ~ 0
+PE4
+Text Label 5400 2400 0    50   ~ 0
+SPI4_SS
+Text Label 1300 2050 2    50   ~ 0
+SPI1_SS
+Text Label 1300 1850 2    50   ~ 0
+SPI4_SS
+Text Label 1900 1450 0    50   ~ 0
+UART2_TX
+Text Label 3575 1700 2    50   ~ 0
+SPI1_SS
+Text Label 3875 1700 0    50   ~ 0
+SPI4_SS
+NoConn ~ 6050 4100
+NoConn ~ 6050 7200
+NoConn ~ 1725 7200
+NoConn ~ 1725 4100
 $EndSCHEMATC

Commit message: clarify schematic
Connections:
- net labels removed: BOOT0, NC, NRST, PA0, PA1, PA13, PA14, PA15, PA6, PA8, PB0, PB1, PB12, PB13, PB14, PB15, PB2, PB3, PB5, PB6, PB9, PC0, PC1, PC13, PC14, PC15, PC2, PC3, PC4, PC5, PC6, PC7, PD0, PD1, PD10, PD11, PD12, PD13, PD14, PD15, PD3, PD4, PD5, PD6, PD7, PD8, PD9, PE0, PE1, PE10, PE11, PE12, PE13, PE14, PE15, PE3, PE7, PE8, PE9, PF0, PF1, PF10, PF11, PF12, PF13, PF14, PF15, PF2, PF3, PF4, PF5, PF6, PF7, PF8, PF9, PG0, PG1, PG10, PG11, PG12, PG13, PG14, PG15, PG2, PG3, PG4, PG5, PG6, PG7, PG8, PG9, PH0, PH1, VDD
- wire segments 36 -> 115
- no-connect marks 4 -> 113
Other:
- note added: "1.1"
- note added: "CSEP Flatsat : STM32F429IDISCOVERY Hat"
- note added: "Connections"
- note added: "Connectors"
- note added: "July 2020"
- note added: "Peripherals"
- note added: "Reference pinout"
- note added: "STM32F429IDISCOVERY headers"
- moved on the sheet: D1, D2, J1, J2, J3, R1, R2, stm32101A, stm32101B

Commit message: Redo routing
Connections:
- net labels removed: I2C2_SDL, SDIO_CK, SDIO_CMD
- wire segments 115 -> 117
- no-connect marks 113 -> 111
Changed lines of the file:
@@
 	8400 4950 8600 4950
 Text Label 8600 4950 0    50   ~ 0
-SDIO_CMD
+SD_CMD
 Wire Wire Line
 	8400 5050 8600 5050
 Text Label 8600 5050 0    50   ~ 0
-SDIO_CK
+SD_CLK
 Text Label 1800 3575 2    50   ~ 0
 I2C1_SDA
@@
 Text Label 4850 3300 2    50   ~ 0
 I2C1_SCL
-Text Label 6175 3125 0    50   ~ 0
+Text Label 6150 3300 0    50   ~ 0
 I2C2_SDA
-Text Label 6175 3225 0    50   ~ 0
-I2C2_SDL
+Text Label 6150 3400 0    50   ~ 0
+I2C2_SCL
 Text Label 4850 3200 2    50   ~ 0
 SPI1_SCK
@@
 Text Label 4850 3000 2    50   ~ 0
 SPI1_MOSI
-Text Label 6175 2825 0    50   ~ 0
+Text Label 6150 3000 0    50   ~ 0
 SPI4_SCK
-Text Label 6175 2925 0    50   ~ 0
+Text Label 6150 3100 0    50   ~ 0
 SPI4_MISO
-Text Label 6175 3025 0    50   ~ 0
+Text Label 6150 3200 0    50   ~ 0
 SPI4_MOSI
 Wire Wire Line
@@
 Text Label 1800 2575 2    50   ~ 0
 UART1_TX
-Text Label 6175 2525 0    50   ~ 0
+Text Label 6150 2700 0    50   ~ 0
 UART1_RX
-Text Label 6175 2625 0    50   ~ 0
+Text Label 6150 2800 0    50   ~ 0
 UART1_TX
 $Comp
@@
 Text Label 4850 2900 2    50   ~ 0
 SPI1_SS
-Text Label 6175 2725 0    50   ~ 0
+Text Label 6150 2900 0    50   ~ 0
 SPI4_SS
-NoConn ~ 5700 7000
 NoConn ~ 5700 10100
 Text Label 1625 6975 2    50   ~ 0
@@
 Text Label 4200 8400 2    50   ~ 0
 GND
-Text Label 4200 7000 2    50   ~ 0
-VCC3
 Text Label 4200 10100 2    50   ~ 0
 GND
@@
 NoConn ~ 5700 9900
 NoConn ~ 5700 10000
-NoConn ~ 5350 2200
 NoConn ~ 5350 2300
 NoConn ~ 5350 2400
-NoConn ~ 5650 2200
 NoConn ~ 5650 2300
 NoConn ~ 5650 2400
@@
 	4200 7900 4700 7900
 Wire Wire Line
-	4200 7000 4700 7000
-Wire Wire Line
 	5700 7900 6200 7900
 Wire Wire Line
@@
 Text Notes 15475 11050 0    50   ~ 0
 1.1
+Text Label 12925 7775 0    50   ~ 0
+GND
+NoConn ~ 5700 7000
+Wire Wire Line
+	4200 7000 4700 7000
+Text Label 4200 7000 2    50   ~ 0
+VCC3
+Text Label 4850 2200 2    50   ~ 0
+VCC
+Text Label 6150 2200 0    50   ~ 0
+GND
+Wire Wire Line
+	4850 2200 5350 2200
+Wire Wire Line
+	6150 2200 5650 2200
 $EndSCHEMATC

Commit message: improve schematic and replace footprints
Parts:
- added JP1: Jumper_2_Bridged, Connector_PinHeader_2.54mm:PinHeader_1x02_P2.54mm_Vertical, symbol Jumper:Jumper_2_Bridged
Connections:
- net labels added: 5V
- net labels removed: PA10, PA11, PA12, PA2, PA3, PA4, PA5, PA7, PA9, PB10, PB11, PB4, PB7, PB8, PC10, PC11, PC12, PC8, PC9, PD2, PE2, PE4, PE5, PE6, SD_DETA, SD_DETB, SD_VDD, SD_VSS, VCC3, VCC5
- wire segments 117 -> 87
- no-connect marks 111 -> 105
Other:
- note added: "1.2"
- note removed: "1.1"
- note removed: "Connections"
- moved on the sheet: D1, D2, J2, R1, R2, stm32101A, stm32101B

Commit message: Replaced DB 26 HD footprint, cleaned layout and few fixes...
Signed-off-by: Alexis Jeandet <alexis.jeandet@member.fsf.org>
Parts:
- added H1, H2, H3, H4: MountingHole_Pad, MountingHole:MountingHole_2.2mm_M2_Pad, symbol Mechanical:MountingHole_Pad
- J1: footprint Connector_Dsub:DSUB-26-HD_Male_Horizontal_P2.29x1.98mm_EdgePinOffset8.35mm_Housed_MountingHolesOffset10.89mm -> DB-HD-26:DSUB-26-HD_Male_Horizontal_P2.29x1.98mm_EdgePinOffset8.35mm_Housed_MountingHolesOffset10.89mm
- J2: footprint Connector_Card:microSD_HC_Hirose_DM3D-SF -> Connector_Card:microSD_HC_Hirose_DM3AT-SF-PEJM5
Connections:
- wire segments 87 -> 92
- no-connect marks 105 -> 104
Changed lines of the file:
@@
 F 0 "J2" H 13500 8092 50  0000 C CNN
 F 1 "Micro_SD_Card_Det" H 13500 8001 50  0000 C CNN
-F 2 "Connector_Card:microSD_HC_Hirose_DM3D-SF" H 15600 7975 50  0001 C CNN
+F 2 "Connector_Card:microSD_HC_Hirose_DM3AT-SF-PEJM5" H 15600 7975 50  0001 C CNN
 F 3 "https://www.hirose.com/product/en/download_file/key_name/DM3/category/Catalog/doc_file_id/49662/?file_category_id=4&item_id=195&is_series=1" H 13550 7375 50  0001 C CNN
 	1    13550 7275
@@
 	12150 7775 12650 7775
 Wire Wire Line
-	14350 7775 14850 7775
+	14350 7775 14825 7775
 Text Label 12150 7775 2    50   ~ 0
 SD_DET
@@
 F 0 "J1" H 11250 4542 50  0000 C CNN
 F 1 "DB26_Male_HighDensity_MountingHoles" H 11250 4451 50  0000 C CNN
-F 2 "Connector_Dsub:DSUB-26-HD_Male_Horizontal_P2.29x1.98mm_EdgePinOffset8.35mm_Housed_MountingHolesOffset10.89mm" H 10300 3325 50  0001 C CNN
+F 2 "DB-HD-26:DSUB-26-HD_Male_Horizontal_P2.29x1.98mm_EdgePinOffset8.35mm_Housed_MountingHolesOffset10.89mm" H 10300 3325 50  0001 C CNN
 F 3 "https://www.mouser.fr/ProductDetail/Kycon/K66X-A26P-N?qs=SY6bF4iPirTxWgCH5IfY4Q%3D%3D" H 10300 3325 50  0001 C CNN
 	1    11250 2925
@@
 NoConn ~ 14300 2250
 NoConn ~ 14300 2350
-NoConn ~ 10950 1825
 NoConn ~ 10950 1925
 NoConn ~ 10950 2025
@@
 L power:GND #PWR0104
 U 1 1 5F3856D8
-P 14850 7775
-F 0 "#PWR0104" H 14850 7525 50  0001 C CNN
-F 1 "GND" H 14855 7602 50  0000 C CNN
-F 2 "" H 14850 7775 50  0001 C CNN
-F 3 "" H 14850 7775 50  0001 C CNN
-	1    14850 7775
+P 14825 7775
+F 0 "#PWR0104" H 14825 7525 50  0001 C CNN
+F 1 "GND" H 14830 7602 50  0000 C CNN
+F 2 "" H 14825 7775 50  0001 C CNN
+F 3 "" H 14825 7775 50  0001 C CNN
+	1    14825 7775
 	1    0    0    -1
 $EndComp
@@
 	0    -1   -1   0
 $EndComp
+$Comp
+L power:VCC #PWR0114
+U 1 1 5F180B31
+P 10850 1825
+F 0 "#PWR0114" H 10850 1675 50  0001 C CNN
+F 1 "VCC" V 10867 1953 50  0000 L CNN
+F 2 "" H 10850 1825 50  0001 C CNN
+F 3 "" H 10850 1825 50  0001 C CNN
+	1    10850 1825
+	0    -1   -1   0
+$EndComp
+Wire Wire Line
+	10850 1825 10950 1825
+$Comp
+L Mechanical:MountingHole_Pad H1
+U 1 1 5F1A4ECB
+P 7950 9675
+F 0 "H1" H 8050 9724 50  0000 L CNN
+F 1 "MountingHole_Pad" H 8050 9633 50  0000 L CNN
+F 2 "MountingHole:MountingHole_2.2mm_M2_Pad" H 7950 9675 50  0001 C CNN
+F 3 "~" H 7950 9675 50  0001 C CNN
+	1    7950 9675
+	1    0    0    -1
+$EndComp
+$Comp
+L Mechanical:MountingHole_Pad H2
+U 1 1 5F1A9D48
+P 7950 10275
+F 0 "H2" H 8050 10324 50  0000 L CNN
+F 1 "MountingHole_Pad" H 8050 10233 50  0000 L CNN
+F 2 "MountingHole:MountingHole_2.2mm_M2_Pad" H 7950 10275 50  0001 C CNN
+F 3 "~" H 7950 10275 50  0001 C CNN
+	1    7950 10275
+	1    0    0    -1
+$EndComp
+$Comp
+L Mechanical:MountingHole_Pad H3
+U 1 1 5F1B0CDB
+P 9125 9675
+F 0 "H3" H 9225 9724 50  0000 L CNN
+F 1 "MountingHole_Pad" H 9225 9633 50  0000 L CNN
+F 2 "MountingHole:MountingHole_2.2mm_M2_Pad" H 9125 9675 50  0001 C CNN
+F 3 "~" H 9125 9675 50  0001 C CNN
+	1    9125 9675
+	1    0    0    -1
+$EndComp
+$Comp
+L Mechanical:MountingHole_Pad H4
+U 1 1 5F1B0CE5
+P 9125 10275
+F 0 "H4" H 9225 10324 50  0000 L CNN
+F 1 "MountingHole_Pad" H 9225 10233 50  0000 L CNN
+F 2 "MountingHole:MountingHole_2.2mm_M2_Pad" H 9125 10275 50  0001 C CNN
+F 3 "~" H 9125 10275 50  0001 C CNN
+	1    9125 10275
+	1    0    0    -1
+$EndComp
+$Comp
+L power:GND #PWR08
+U 1 1 5F1B8016
+P 7950 10475
+F 0 "#PWR08" H 7950 10225 50  0001 C CNN
+F 1 "GND" H 7955 10302 50  0000 C CNN
+F 2 "" H 7950 10475 50  0001 C CNN
+F 3 "" H 7950 10475 50  0001 C CNN
+	1    7950 10475
+	1    0    0    -1
+$EndComp
+Wire Wire Line
+	7950 10475 7950 10375
+$Comp
+L power:GND #PWR07
+U 1 1 5F1C36E1
+P 7950 9875
+F 0 "#PWR07" H 7950 9625 50  0001 C CNN
+F 1 "GND" H 7955 9702 50  0000 C CNN
+F 2 "" H 7950 9875 50  0001 C CNN
+F 3 "" H 7950 9875 50  0001 C CNN
+	1    7950 9875
+	1    0    0    -1
+$EndComp
+Wire Wire Line
+	7950 9875 7950 9775
+$Comp
+L power:GND #PWR09
+U 1 1 5F1D16E2
+P 9125 9875
+F 0 "#PWR09" H 9125 9625 50  0001 C CNN
+F 1 "GND" H 9130 9702 50  0000 C CNN
+F 2 "" H 9125 9875 50  0001 C CNN
+F 3 "" H 9125 9875 50  0001 C CNN
+	1    9125 9875
+	1    0    0    -1
+$EndComp
+Wire Wire Line
+	9125 9875 9125 9775
+$Comp
+L power:GND #PWR010
+U 1 1 5F1D62FA
+P 9125 10475
+F 0 "#PWR010" H 9125 10225 50  0001 C CNN
+F 1 "GND" H 9130 10302 50  0000 C CNN
+F 2 "" H 9125 10475 50  0001 C CNN
+F 3 "" H 9125 10475 50  0001 C CNN
+	1    9125 10475
+	1    0    0    -1
+$EndComp
+Wire Wire Line
+	9125 10475 9125 10375
 $EndSCHEMATC
